File: psu_4caps.sch (KiCad schematic (older format))
At the start: 37 parts, among them J1 AC1, J10 GND, J11 V-, J12 V-, J2 GND2, J3 GND3, J4 AC4, J5 LED, J6 LED, J7 V+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

Commit message: finished pcb layout
Parts:
- added H5: MountingHole, MountingHole:MountingHole_3.2mm_M3_Pad_Via, symbol Mechanical:MountingHole
- C10, C7, C8, C9: footprint Capacitor_THT:CP_Radial_D25.0mm_P10.00mm_SnapIn -> Capacitor_THT:CP_Radial_D35.0mm_P10.00mm_SnapIn
Changed lines of the file:
@@
 F 0 "C7" H 4588 3546 50  0000 L CNN
 F 1 "22,000u" H 4588 3455 50  0000 L CNN
-F 2 "Capacitor_THT:CP_Radial_D25.0mm_P10.00mm_SnapIn" H 4500 3500 50  0001 C CNN
+F 2 "Capacitor_THT:CP_Radial_D35.0mm_P10.00mm_SnapIn" H 4500 3500 50  0001 C CNN
 F 3 "~" H 4500 3500 50  0001 C CNN
 	1    4500 3500
@@
 F 0 "C9" H 5138 3546 50  0000 L CNN
 F 1 "22,000u" H 5138 3455 50  0000 L CNN
-F 2 "Capacitor_THT:CP_Radial_D25.0mm_P10.00mm_SnapIn" H 5050 3500 50  0001 C CNN
+F 2 "Capacitor_THT:CP_Radial_D35.0mm_P10.00mm_SnapIn" H 5050 3500 50  0001 C CNN
 F 3 "~" H 5050 3500 50  0001 C CNN
 	1    5050 3500
@@
 F 0 "C8" H 4588 4546 50  0000 L CNN
 F 1 "22,000u" H 4588 4455 50  0000 L CNN
-F 2 "Capacitor_THT:CP_Radial_D25.0mm_P10.00mm_SnapIn" H 4500 4500 50  0001 C CNN
+F 2 "Capacitor_THT:CP_Radial_D35.0mm_P10.00mm_SnapIn" H 4500 4500 50  0001 C CNN
 F 3 "~" H 4500 4500 50  0001 C CNN
 	1    4500 4500
@@
 F 0 "C10" H 5138 4546 50  0000 L CNN
 F 1 "22,000u" H 5138 4455 50  0000 L CNN
-F 2 "Capacitor_THT:CP_Radial_D25.0mm_P10.00mm_SnapIn" H 5050 4500 50  0001 C CNN
+F 2 "Capacitor_THT:CP_Radial_D35.0mm_P10.00mm_SnapIn" H 5050 4500 50  0001 C CNN
 F 3 "~" H 5050 4500 50  0001 C CNN
 	1    5050 4500
@@
 Wire Wire Line
 	5050 4000 5650 4000
+$Comp
+L Mechanical:MountingHole H5
+U 1 1 65A5C1F9
+P 1500 7000
+F 0 "H5" H 1600 7046 50  0000 L CNN
+F 1 "MountingHole" H 1600 6955 50  0000 L CNN
+F 2 "MountingHole:MountingHole_3.2mm_M3_Pad_Via" H 1500 7000 50  0001 C CNN
+F 3 "~" H 1500 7000 50  0001 C CNN
+	1    1500 7000
+	1    0    0    -1
+$EndComp
 $EndSCHEMATC

Commit message: rev2 commit
Parts:
- added J13: AUX OUT, local_footprints_lib:TerminalBlock_ Amphenol_01_03_P3.50mm, symbol Connector:Screw_Terminal_01x03
- C3, C4, C5, C6: footprint Capacitor_THT:C_Rect_L7.2mm_W2.5mm_P5.00mm_FKS2_FKP2_MKS2_MKP2 -> Capacitor_THT:C_Rect_L7.2mm_W4.5mm_P5.00mm_FKS2_FKP2_MKS2_MKP2
- D2, D3: value LED -> LED_SMD; footprint Diode_SMD:D_0805_2012Metric_Pad1.15x1.40mm_HandSolder -> LED_SMD:LED_0805_2012Metric_Pad1.15x1.40mm_HandSolder; Field4 SMD -> (none)
- R3, R4: footprint Resistor_THT:R_Axial_DIN0207_L6.3mm_D2.5mm_P10.16mm_Horizontal -> Resistor_SMD:R_1206_3216Metric_Pad1.42x1.75mm_HandSolder
- R5, R6: value 10K -> 47K; footprint Resistor_THT:R_Axial_DIN0207_L6.3mm_D2.5mm_P10.16mm_Horizontal -> Resistor_SMD:R_1206_3216Metric_Pad1.42x1.75mm_HandSolder
Connections:
- net GND: now also D2.1 (K), J13.2 (Pin_2); no longer D2.2 (A)
- net V+: now also J13.1 (Pin_1)
- net V-: now also D3.1 (K), J13.3 (Pin_3); no longer D3.2 (A)
- net at R5.2: now also D2.2 (A); no longer D2.1 (K)
- net at R6.2: now also D3.2 (A); no longer D3.1 (K)
Changed lines of the file:
@@
 	6150 4000 6700 4000
-$Comp
-L Device:LED_Small D2
-U 1 1 64A76D0F
-P 6700 3750
-F 0 "D2" V 6609 3848 50  0000 L CNN
-F 1 "LED" V 6700 3848 50  0000 L CNN
-F 2 "Diode_SMD:D_0805_2012Metric_Pad1.15x1.40mm_HandSolder" V 6700 3750 50  0001 C CNN
-F 3 "~" V 6700 3750 50  0001 C CNN
-F 4 "SMD" V 6791 3848 50  0000 L CNN "Field4"
-	1    6700 3750
-	0    1    1    0
-$EndComp
 $Comp
 L Device:R_Small R5
@@
 P 6700 3250
 F 0 "R5" H 6759 3296 50  0000 L CNN
-F 1 "10K" H 6759 3205 50  0000 L CNN
-F 2 "Resistor_THT:R_Axial_DIN0207_L6.3mm_D2.5mm_P10.16mm_Horizontal" H 6700 3250 50  0001 C CNN
+F 1 "47K" H 6759 3205 50  0000 L CNN
+F 2 "Resistor_SMD:R_1206_3216Metric_Pad1.42x1.75mm_HandSolder" H 6700 3250 50  0001 C CNN
 F 3 "~" H 6700 3250 50  0001 C CNN
 	1    6700 3250
 	1    0    0    -1
-$EndComp
-$Comp
-L Device:LED_Small D3
-U 1 1 64A8796E
-P 6700 4750
-F 0 "D3" V 6609 4848 50  0000 L CNN
-F 1 "LED" V 6700 4848 50  0000 L CNN
-F 2 "Diode_SMD:D_0805_2012Metric_Pad1.15x1.40mm_HandSolder" V 6700 4750 50  0001 C CNN
-F 3 "~" V 6700 4750 50  0001 C CNN
-F 4 "SMD" V 6791 4848 50  0000 L CNN "Field4"
-	1    6700 4750
-	0    1    1    0
 $EndComp
 Wire Wire Line
@@
 F 0 "R3" H 6209 3296 50  0000 L CNN
 F 1 "10K" H 6209 3205 50  0000 L CNN
-F 2 "Resistor_THT:R_Axial_DIN0207_L6.3mm_D2.5mm_P10.16mm_Horizontal" H 6150 3250 50  0001 C CNN
+F 2 "Resistor_SMD:R_1206_3216Metric_Pad1.42x1.75mm_HandSolder" H 6150 3250 50  0001 C CNN
 F 3 "~" H 6150 3250 50  0001 C CNN
 	1    6150 3250
@@
 F 0 "R4" H 6209 4296 50  0000 L CNN
 F 1 "10K" H 6209 4205 50  0000 L CNN
-F 2 "Resistor_THT:R_Axial_DIN0207_L6.3mm_D2.5mm_P10.16mm_Horizontal" H 6150 4250 50  0001 C CNN
+F 2 "Resistor_SMD:R_1206_3216Metric_Pad1.42x1.75mm_HandSolder" H 6150 4250 50  0001 C CNN
 F 3 "~" H 6150 4250 50  0001 C CNN
 	1    6150 4250
@@
 P 6700 4250
 F 0 "R6" H 6759 4296 50  0000 L CNN
-F 1 "10K" H 6759 4205 50  0000 L CNN
-F 2 "Resistor_THT:R_Axial_DIN0207_L6.3mm_D2.5mm_P10.16mm_Horizontal" H 6700 4250 50  0001 C CNN
+F 1 "47K" H 6759 4205 50  0000 L CNN
+F 2 "Resistor_SMD:R_1206_3216Metric_Pad1.42x1.75mm_HandSolder" H 6700 4250 50  0001 C CNN
 F 3 "~" H 6700 4250 50  0001 C CNN
 	1    6700 4250
@@
 F 0 "C3" H 2892 3696 50  0000 L CNN
 F 1 "100n" H 2892 3605 50  0000 L CNN
-F 2 "Capacitor_THT:C_Rect_L7.2mm_W2.5mm_P5.00mm_FKS2_FKP2_MKS2_MKP2" H 2800 3650 50  0001 C CNN
+F 2 "Capacitor_THT:C_Rect_L7.2mm_W4.5mm_P5.00mm_FKS2_FKP2_MKS2_MKP2" H 2800 3650 50  0001 C CNN
 F 3 "~" H 2800 3650 50  0001 C CNN
 F 4 "film" H 3000 3500 50  0000 C CNN "Field4"
@@
 F 0 "C4" H 2892 4346 50  0000 L CNN
 F 1 "100n" H 2892 4255 50  0000 L CNN
-F 2 "Capacitor_THT:C_Rect_L7.2mm_W2.5mm_P5.00mm_FKS2_FKP2_MKS2_MKP2" H 2800 4300 50  0001 C CNN
+F 2 "Capacitor_THT:C_Rect_L7.2mm_W4.5mm_P5.00mm_FKS2_FKP2_MKS2_MKP2" H 2800 4300 50  0001 C CNN
 F 3 "~" H 2800 4300 50  0001 C CNN
 F 4 "film" H 3000 4150 50  0000 C CNN "Field4"
@@
 F 0 "C5" H 3892 3696 50  0000 L CNN
 F 1 "100n" H 3892 3605 50  0000 L CNN
-F 2 "Capacitor_THT:C_Rect_L7.2mm_W2.5mm_P5.00mm_FKS2_FKP2_MKS2_MKP2" H 3800 3650 50  0001 C CNN
+F 2 "Capacitor_THT:C_Rect_L7.2mm_W4.5mm_P5.00mm_FKS2_FKP2_MKS2_MKP2" H 3800 3650 50  0001 C CNN
 F 3 "~" H 3800 3650 50  0001 C CNN
 F 4 "film" H 4000 3500 50  0000 C CNN "Field4"
@@
 F 0 "C6" H 3892 4346 50  0000 L CNN
 F 1 "100n" H 3892 4255 50  0000 L CNN
-F 2 "Capacitor_THT:C_Rect_L7.2mm_W2.5mm_P5.00mm_FKS2_FKP2_MKS2_MKP2" H 3800 4300 50  0001 C CNN
+F 2 "Capacitor_THT:C_Rect_L7.2mm_W4.5mm_P5.00mm_FKS2_FKP2_MKS2_MKP2" H 3800 4300 50  0001 C CNN
 F 3 "~" H 3800 4300 50  0001 C CNN
 F 4 "film" H 4000 4150 50  0000 C CNN "Field4"
@@
 	1    0    0    -1
 $EndComp
+$Comp
+L Device:LED_Small D3
+U 1 1 65B19176
+P 6700 4750
+F 0 "D3" V 6746 4680 50  0000 R CNN
+F 1 "LED_SMD" V 6655 4680 50  0000 R CNN
+F 2 "LED_SMD:LED_0805_2012Metric_Pad1.15x1.40mm_HandSolder" V 6700 4750 50  0001 C CNN
+F 3 "~" V 6700 4750 50  0001 C CNN
+	1    6700 4750
+	0    -1   -1   0
+$EndComp
+$Comp
+L Device:LED_Small D2
+U 1 1 65B1BDEB
+P 6700 3750
+F 0 "D2" V 6746 3680 50  0000 R CNN
+F 1 "LED_SMD" V 6655 3680 50  0000 R CNN
+F 2 "LED_SMD:LED_0805_2012Metric_Pad1.15x1.40mm_HandSolder" V 6700 3750 50  0001 C CNN
+F 3 "~" V 6700 3750 50  0001 C CNN
+	1    6700 3750
+	0    -1   -1   0
+$EndComp
+$Comp
+L Connector:Screw_Terminal_01x03 J13
+U 1 1 65B4ABFD
+P 7450 5500
+F 0 "J13" H 7530 5542 50  0000 L CNN
+F 1 "AUX OUT" H 7530 5451 50  0000 L CNN
+F 2 "local_footprints_lib:TerminalBlock_ Amphenol_01_03_P3.50mm" H 7450 5500 50  0001 C CNN
+F 3 "~" H 7450 5500 50  0001 C CNN
+	1    7450 5500
+	1    0    0    -1
+$EndComp
+$Comp
+L power:GND #PWR05
+U 1 1 65B51662
+P 7050 5500
+F 0 "#PWR05" H 7050 5250 50  0001 C CNN
+F 1 "GND" H 7055 5327 50  0001 C CNN
+F 2 "" H 7050 5500 50  0001 C CNN
+F 3 "" H 7050 5500 50  0001 C CNN
+	1    7050 5500
+	1    0    0    -1
+$EndComp
+Wire Wire Line
+	7050 5500 7250 5500
+Text Label 7050 5700 0    50   ~ 0
+V-
+Text Label 7050 5350 0    50   ~ 0
+V+
+Wire Wire Line
+	7250 5400 7050 5400
+Wire Wire Line
+	7050 5400 7050 5350
+Wire Wire Line
+	7250 5600 7200 5600
+Wire Wire Line
+	7200 5600 7200 5700
+Wire Wire Line
+	7200 5700 7050 5700
 $EndSCHEMATC
